Commit message: robot finally is added

File: lab2andDriver/drivers/universal_robot/ur_description/urdf/ur3.urdf (robot description, URDF)
Before this commit: robot ur3, 15 links, 14 joints
Links:
- removed link cart_chassis_link
- removed link left_wheel
- removed link right_wheel
Joints:
- removed joint cart_chassis_fixed
- removed joint left_wheel_hinge
- removed joint right_wheel_hinge

File: lab2andDriver/drivers/universal_robot/ur_description/urdf/ur3_robot.urdf.xacro (robot description, xacro)
@@ -7,13 +7,14 @@
   <!-- ur3 -->
   <xacro:include filename="$(find ur_description)/urdf/ur3.urdf.xacro" />
+  <!-- cartopole -->
+  <xacro:include filename="$(find ur_description)/urdf/myrobot.xacro" />
   <!-- arm -->
   <xacro:ur3_robot prefix="" joint_limited="false"
     transmission_hw_interface="$(arg transmission_hw_interface)"
   />
-  <link name="world" />
-  <joint name="world_joint" type="fixed">
-    <parent link="world" />
+  <joint name="ur3_cart_joint" type="fixed">
+    <parent link="chassis" />
     <child link = "base_link" />
-    <origin xyz="0.0 0.0 0.0" rpy="0.0 0.0 0.0" />
+    <origin xyz="0.0 0.0 0.05" rpy="0.0 0.0 0.0" />
   </joint>
 </robot>
