Commit message: idk if this is working but trying another way

File: lab2andDriver/drivers/universal_robot/ur_description/urdf/macros.xacro (robot description, xacro)
@@ -1,23 +1,23 @@
 <?xml version="1.0"?>
 <robot>
-  <macro name="cylinder_inertia" params="m r h">
+  <xacro:macro name="cylinder_inertia" params="m r h">
     <inertia  ixx="${m*(3*r*r+h*h)/12}" ixy = "0" ixz = "0"
       iyy="${m*(3*r*r+h*h)/12}" iyz = "0"
       izz="${m*r*r/2}"
     />
-  </macro>
-  <macro name="box_inertia" params="m x y z">
+  </xacro:macro>
+  <xacro:macro name="box_inertia" params="m x y z">
     <inertia  ixx="${m*(y*y+z*z)/12}" ixy = "0" ixz = "0"
       iyy="${m*(x*x+z*z)/12}" iyz = "0"
       izz="${m*(x*x+z*z)/12}"
     />
-  </macro>
-  <macro name="sphere_inertia" params="m r">
+  </xacro:macro>
+  <xacro:macro name="sphere_inertia" params="m r">
     <inertia  ixx="${2*m*r*r/5}" ixy = "0" ixz = "0"
       iyy="${2*m*r*r/5}" iyz = "0"
       izz="${2*m*r*r/5}"
     />
-  </macro>
-  <macro name="wheel" params="lr tY">
+  </xacro:macro>
+  <xacro:macro name="wheel" params="lr tY">
     <link name="${lr}_wheel">
       <collision>
@@ -66,4 +66,4 @@
       </actuator>
     </transmission>
-  </macro>
+  </xacro:macro>
 </robot>

File: lab2andDriver/drivers/universal_robot/ur_description/urdf/myrobot.xacro (robot description, xacro)
@@ -1,125 +1,172 @@
 <?xml version='1.0'?>
-<robot name="robot" xmlns:xacro="http://www.ros.org/wiki/xacro">
-  <xacro:include filename="$(find ur_description)/urdf/myrobot.gazebo" />
-  <xacro:include filename="$(find ur_description)/urdf/materials.xacro" />
-  <xacro:include filename="$(find ur_description)/urdf/macros.xacro" />
-  <link name='chassis'>
-    <pose>0 0 0.1 0 0 0</pose>
-    <inertial>
-      <mass value="10.0"/>
-      <origin xyz="0.0 0 0.1" rpy=" 0 0 0"/>
-      <inertia
-          ixx="0.5" ixy="0" ixz="0"
-          iyy="1.0" iyz="0"
-          izz="0.1"
-      />
-    </inertial>
-    <collision name='collision'>
-      <geometry>
-        <box size=".4 .2 .1"/>
-      </geometry>
-    </collision>
-    <visual name='chassis_visual'>
-      <origin xyz="0 0 0" rpy=" 0 0 0"/>
-      <geometry>
-        <box size=".4 .2 .1"/>
-      </geometry>
-    </visual>
-    <collision name='caster_collision'>
-      <origin xyz="-0.15 0 -0.05" rpy=" 0 0 0"/>
-      <geometry>
-        <sphere radius="0.05"/>
-      </geometry>
-    </collision>
-    <visual name='caster_visual'>
-      <origin xyz="-0.15 0 -0.05" rpy=" 0 0 0"/>
-      <geometry>
-        <sphere radius="0.05"/>
-      </geometry>
-    </visual>
-  </link>
-  <link name="left_wheel">
-    <!--origin xyz="0.1 0.13 0.1" rpy="0 1.5707 1.5707"/-->
-    <collision name="collision">
-      <origin xyz="0 0 0" rpy="0 1.5707 1.5707"/>
-      <geometry>
-        <cylinder radius="0.1" length="0.05"/>
-      </geometry>
-    </collision>
-    <visual name="left_wheel_visual">
-      <origin xyz="0 0 0" rpy="0 1.5707 1.5707"/>
-      <geometry>
-        <cylinder radius="0.1" length="0.05"/>
-      </geometry>
-    </visual>
-    <inertial>
-      <origin xyz="0 0 0" rpy="0 1.5707 1.5707"/>
-      <mass value="5"/>
-      <cylinder_inertia m="5" r="0.1" h="0.05"/>
-      <inertia
-        ixx="1.0" ixy="0.0" ixz="0.0"
-        iyy="1.0" iyz="0.0"
-        izz="1.0"/>
-    </inertial>
-  </link>
-  <link name="right_wheel">
-    <!--origin xyz="0.1 -0.13 0.1" rpy="0 1.5707 1.5707"/-->
-    <collision name="collision">
-      <origin xyz="0 0 0" rpy="0 1.5707 1.5707"/>
-      <geometry>
-        <cylinder radius="0.1" length="0.05"/>
-      </geometry>
-    </collision>
-    <visual name="right_wheel_visual">
-      <origin xyz="0 0 0" rpy="0 1.5707 1.5707"/>
-      <geometry>
-        <cylinder radius="0.1" length="0.05"/>
-      </geometry>
-    </visual>
-    <inertial>
-      <origin xyz="0 0 0" rpy="0 1.5707 1.5707"/>
-      <mass value="5"/>
-      <cylinder_inertia m="5" r="0.1" h="0.05"/>
-      <inertia
-        ixx="1.0" ixy="0.0" ixz="0.0"
-        iyy="1.0" iyz="0.0"
-        izz="1.0"/>
-    </inertial>
-  </link>
-  <joint type="continuous" name="left_wheel_hinge">
-    <origin xyz="0.1 0.15 0" rpy="0 0 0"/>
-    <child link="left_wheel"/>
-    <parent link="chassis"/>
-    <axis xyz="0 1 0" rpy="0 0 0"/>
-    <!-- <limit velocity="100"/> -->
-    <joint_properties damping="0.0" friction="0.0"/>
-  </joint>
-  <joint type="continuous" name="right_wheel_hinge">
-    <origin xyz="0.1 -0.15 0" rpy="0 0 0"/>
-    <child link="right_wheel"/>
-    <parent link="chassis"/>
-    <axis xyz="0 1 0" rpy="0 0 0"/>
-    <!-- <limit velocity="100"/> -->
-    <joint_properties damping="0.0" friction="0.0"/>
-  </joint>
-  <transmission name="left_trans">
-      <type>transmission_interface/SimpleTransmission</type>
-      <joint name="left_wheel_hinge">
-        <hardwareInterface>EffortJointInterface</hardwareInterface>
-      </joint>
-      <actuator name="leftMotor">
-        <hardwareInterface>EffortJointInterface</hardwareInterface>
-        <mechanicalReduction>10</mechanicalReduction>
-      </actuator>
-    </transmission>
-    <transmission name="right_trans">
-      <type>transmission_interface/SimpleTransmission</type>
-      <joint name="right_wheel_hinge">
-        <hardwareInterface>EffortJointInterface</hardwareInterface>
-      </joint>
-      <actuator name="rightMotor">
-        <hardwareInterface>EffortJointInterface</hardwareInterface>
-        <mechanicalReduction>10</mechanicalReduction>
-      </actuator>
-    </transmission>
+<robot xmlns:xacro="http://www.ros.org/wiki/xacro">
+  <!-- <xacro:include filename="$(find ur_description)/urdf/myrobot.gazebo" /> -->
+  <!-- <xacro:include filename="$(find ur_description)/urdf/materials.xacro" /> -->
+  <!-- <xacro:include filename="$(find ur_description)/urdf/macros.xacro" /> -->
+  <xacro:macro name="cart_robot">
+    <link name='chassis'>
+      <pose>0 0 0.1 0 0 0</pose>
+      <inertial>
+        <mass value="10.0"/>
+        <origin xyz="0.0 0 0.1" rpy=" 0 0 0"/>
+        <inertia
+            ixx="0.5" ixy="0" ixz="0"
+            iyy="1.0" iyz="0"
+            izz="0.1"
+        />
+      </inertial>
+      <collision name='collision'>
+        <geometry>
+          <box size=".4 .2 .1"/>
+        </geometry>
+      </collision>
+      <visual name='chassis_visual'>
+        <origin xyz="0 0 0" rpy=" 0 0 0"/>
+        <geometry>
+          <box size=".4 .2 .1"/>
+        </geometry>
+      </visual>
+      <collision name='caster_collision'>
+        <origin xyz="-0.15 0 -0.05" rpy=" 0 0 0"/>
+        <geometry>
+          <sphere radius="0.05"/>
+        </geometry>
+      </collision>
+      <visual name='caster_visual'>
+        <origin xyz="-0.15 0 -0.05" rpy=" 0 0 0"/>
+        <geometry>
+          <sphere radius="0.05"/>
+        </geometry>
+      </visual>
+    </link>
+    <link name="left_wheel">
+      <!--origin xyz="0.1 0.13 0.1" rpy="0 1.5707 1.5707"/-->
+      <collision name="collision">
+        <origin xyz="0 0 0" rpy="0 1.5707 1.5707"/>
+        <geometry>
+          <cylinder radius="0.1" length="0.05"/>
+        </geometry>
+      </collision>
+      <visual name="left_wheel_visual">
+        <origin xyz="0 0 0" rpy="0 1.5707 1.5707"/>
+        <geometry>
+          <cylinder radius="0.1" length="0.05"/>
+        </geometry>
+      </visual>
+      <inertial>
+        <origin xyz="0 0 0" rpy="0 1.5707 1.5707"/>
+        <mass value="5"/>
+        <cylinder_inertia m="5" r="0.1" h="0.05"/>
+        <inertia
+          ixx="1.0" ixy="0.0" ixz="0.0"
+          iyy="1.0" iyz="0.0"
+          izz="1.0"/>
+      </inertial>
+    </link>
+    <link name="right_wheel">
+      <!--origin xyz="0.1 -0.13 0.1" rpy="0 1.5707 1.5707"/-->
+      <collision name="collision">
+        <origin xyz="0 0 0" rpy="0 1.5707 1.5707"/>
+        <geometry>
+          <cylinder radius="0.1" length="0.05"/>
+        </geometry>
+      </collision>
+      <visual name="right_wheel_visual">
+        <origin xyz="0 0 0" rpy="0 1.5707 1.5707"/>
+        <geometry>
+          <cylinder radius="0.1" length="0.05"/>
+        </geometry>
+      </visual>
+      <inertial>
+        <origin xyz="0 0 0" rpy="0 1.5707 1.5707"/>
+        <mass value="5"/>
+        <cylinder_inertia m="5" r="0.1" h="0.05"/>
+        <inertia
+          ixx="1.0" ixy="0.0" ixz="0.0"
+          iyy="1.0" iyz="0.0"
+          izz="1.0"/>
+      </inertial>
+    </link>
+    <joint type="continuous" name="left_wheel_hinge">
+      <origin xyz="0.1 0.15 0" rpy="0 0 0"/>
+      <child link="left_wheel"/>
+      <parent link="chassis"/>
+      <axis xyz="0 1 0" rpy="0 0 0"/>
+      <!-- <limit velocity="100"/> -->
+      <joint_properties damping="0.0" friction="0.0"/>
+    </joint>
+    <joint type="continuous" name="right_wheel_hinge">
+      <origin xyz="0.1 -0.15 0" rpy="0 0 0"/>
+      <child link="right_wheel"/>
+      <parent link="chassis"/>
+      <axis xyz="0 1 0" rpy="0 0 0"/>
+      <!-- <limit velocity="100"/> -->
+      <joint_properties damping="0.0" friction="0.0"/>
+    </joint>
+    <transmission name="left_trans">
+        <type>transmission_interface/SimpleTransmission</type>
+        <joint name="left_wheel_hinge">
+          <hardwareInterface>hardware_interface/VelocityJointInterface</hardwareInterface>
+        </joint>
+        <actuator name="leftMotor">
+          <hardwareInterface>VelocityJointInterface</hardwareInterface>
+          <mechanicalReduction>10</mechanicalReduction>
+        </actuator>
+      </transmission>
+      <transmission name="right_trans">
+        <type>transmission_interface/SimpleTransmission</type>
+        <joint name="right_wheel_hinge">
+          <hardwareInterface>hardware_interface/VelocityJointInterface</hardwareInterface>
+        </joint>
+        <actuator name="rightMotor">
+          <hardwareInterface>VelocityJointInterface</hardwareInterface>
+          <mechanicalReduction>10</mechanicalReduction>
+        </actuator>
+      </transmission>
+    <gazebo>
+      <plugin name="differential_drive_controller" filename="libgazebo_ros_diff_drive.so">
+        <robotNamespace>/differential_drive</robotNamespace>
+        <legacyMode>True</legacyMode>
+        <!-- <robotSimType>gazebo_ros_control/DefaultRobotHWSim</robotSimType> -->
+        <alwaysOn>true</alwaysOn>
+        <updateRate>20</updateRate>
+        <leftJoint>left_wheel_hinge</leftJoint>
+        <rightJoint>right_wheel_hinge</rightJoint>
+        <wheelSeparation>0.4</wheelSeparation>
+        <wheelDiameter>0.1</wheelDiameter>
+        <torque>20</torque>
+        <commandTopic>cmd_vel</commandTopic>
+        <odometryTopic>odom</odometryTopic>
+        <odometryFrame>odom</odometryFrame>
+        <robotBaseFrame>chassis</robotBaseFrame>
+        <publishWheelTF>false</publishWheelTF>
+        <publishOdom>false</publishOdom>
+        <publishOdomTF>true</publishOdomTF>
+        <publishWheelJointState>false</publishWheelJointState>
+        <wheelAcceleration>0</wheelAcceleration>
+        <wheelTorque>5</wheelTorque>
+        <odometrySource>world</odometrySource>
+        <publishTf>1</publishTf>
+        <rosDebugLevel>na</rosDebugLevel>
+      </plugin>
+    </gazebo>
+    <gazebo reference="chassis">
+      <selfCollide>true</selfCollide>
+      <mu1>0.0</mu1>
+      <mu2>0.0</mu2>
+      <material>Gazebo/Orange</material>
+    </gazebo>
+    <gazebo reference="left_wheel">
+      <selfCollide>true</selfCollide>
+      <mu1>0.2</mu1>
+      <mu2>0.2</mu2>
+      <material>Gazebo/Black</material>
+    </gazebo>
+    <gazebo reference="right_wheel">
+      <selfCollide>true</selfCollide>
+      <mu1>0.2</mu1>
+      <mu2>0.2</mu2>
+      <material>Gazebo/Black</material>
+    </gazebo>
+  </xacro:macro>
 </robot>

File: lab2andDriver/drivers/universal_robot/ur_description/urdf/ur3.urdf.xacro (robot description, xacro)
@@ -6,5 +6,5 @@
   <xacro:include filename="$(find ur_description)/urdf/ur.transmission.xacro" />
   <xacro:include filename="$(find ur_description)/urdf/ur.gazebo.xacro" />
-   <xacro:macro name="cylinder_inertial" params="radius length mass *origin">
+  <xacro:macro name="cylinder_inertial" params="radius length mass *origin">
     <inertial>
       <mass value="${mass}" />

File: lab2andDriver/drivers/universal_robot/ur_description/urdf/ur3_robot.urdf.xacro (robot description, xacro)
@@ -13,4 +13,5 @@
     transmission_hw_interface="$(arg transmission_hw_interface)"
   />
+  <xacro:cart_robot/>
   <joint name="ur3_cart_joint" type="fixed">
     <parent link="chassis" />
