Commit message: update 2 final push

File: lab2andDriver/drivers/universal_robot/ur_description/urdf/ur3_robot.urdf.xacro (robot description, xacro)
@@ -13,8 +13,8 @@
     transmission_hw_interface="$(arg transmission_hw_interface)"
   />
-  <joint name="ur3_cart_joint" type="fixed">
+  <!-- <joint name="ur3_cart_joint" type="fixed">
     <parent link="chassis" />
     <child link = "base_link" />
     <origin xyz="0.0 0.0 0.05" rpy="0.0 0.0 0.0" />
-  </joint>
+  </joint> -->
 </robot>

Commit message: implementing lab functions

File: lab2andDriver/drivers/universal_robot/ur_description/urdf/ur3_robot.urdf.xacro (robot description, xacro)
@@ -15,7 +15,7 @@
   <xacro:cart_robot/>
   <joint name="ur3_cart_joint" type="fixed">
-    <parent link="base_link" />
-    <child link = "chassis" />
-    <origin xyz="0.0 0.0 -0.05" rpy="0.0 0.0 0.0" />
+    <parent link="chassis" />
+    <child link = "base_link" />
+    <origin xyz="0.0 0.0 0.05" rpy="0.0 0.0 0.0" />
   </joint>
 </robot>
