Commit message: joint state convergence confirmed'

File: lab2andDriver/drivers/universal_robot/ur_description/urdf/ur3_joint_limited_robot.urdf.xacro (robot description, xacro)
@@ -5,7 +5,9 @@
   <!-- common stuff -->
   <xacro:include filename="$(find ur_description)/urdf/common.gazebo.xacro" />
+  <!-- ur3 macros -->
+  <xacro:include filename="$(find ur_description)/urdf/ur3.urdf.xacro" />
+  <!-- cart macros-->
+  <xacro:include filename="$(find ur_description)/urdf/myrobot.xacro" />
   <!-- ur3 -->
-  <xacro:include filename="$(find ur_description)/urdf/ur3.urdf.xacro" />
-  <!-- arm -->
   <xacro:ur3_robot prefix="" joint_limited="true"
     shoulder_pan_lower_limit="${-pi}" shoulder_pan_upper_limit="${pi}"
@@ -17,9 +19,10 @@
     transmission_hw_interface="$(arg transmission_hw_interface)"
   />
-  <link name="world" />
-  <joint name="world_joint" type="fixed">
-    <parent link="world" />
+  <!-- cart -->
+  <xacro:cart_robot/>
+  <joint name="ur3_cart_joint" type="fixed">
+    <parent link="chassis" />
     <child link = "base_link" />
-    <origin xyz="0.0 0.0 0.0" rpy="0.0 0.0 0.0" />
+    <origin xyz="0.0 0.0 0.05" rpy="0.0 0.0 0.0" />
   </joint>
 </robot>

File: lab2andDriver/drivers/universal_robot/ur_description/urdf/ur3_robot.urdf.xacro (robot description, xacro)
@@ -19,5 +19,4 @@
     <origin xyz="0.0 0.0 0.05" rpy="0.0 0.0 0.0" />
   </joint>
-  <!--
   <link name="world" />
   <joint name="ur3_cart_joint_fix" type="fixed">
@@ -25,4 +24,4 @@
     <child link = "chassis" />
     <origin xyz="0.0 0.0 0.0" rpy="0.0 0.0 0.0" />
-  </joint> -->
+  </joint>
 </robot>
