Commit message: working on getting the contorl file

File: lab2andDriver/drivers/universal_robot/ur_description/urdf/myrobot.xacro (robot description, xacro)
@@ -103,3 +103,23 @@
     <joint_properties damping="0.0" friction="0.0"/>
   </joint>
+  <transmission name="left_trans">
+      <type>transmission_interface/SimpleTransmission</type>
+      <joint name="left_wheel_hinge">
+        <hardwareInterface>EffortJointInterface</hardwareInterface>
+      </joint>
+      <actuator name="leftMotor">
+        <hardwareInterface>EffortJointInterface</hardwareInterface>
+        <mechanicalReduction>10</mechanicalReduction>
+      </actuator>
+    </transmission>
+    <transmission name="right_trans">
+      <type>transmission_interface/SimpleTransmission</type>
+      <joint name="right_wheel_hinge">
+        <hardwareInterface>EffortJointInterface</hardwareInterface>
+      </joint>
+      <actuator name="rightMotor">
+        <hardwareInterface>EffortJointInterface</hardwareInterface>
+        <mechanicalReduction>10</mechanicalReduction>
+      </actuator>
+    </transmission>
 </robot>

Commit message: cart control of robot

File: lab2andDriver/drivers/universal_robot/ur_description/urdf/myrobot.xacro (robot description, xacro)
@@ -126,7 +126,8 @@
     <gazebo>
       <plugin name="differential_drive_controller" filename="libgazebo_ros_diff_drive.so">
-        <robotNamespace>/differential_drive</robotNamespace>
+        <robotNamespace>/cart_controller</robotNamespace>
         <legacyMode>True</legacyMode>
         <!-- <robotSimType>gazebo_ros_control/DefaultRobotHWSim</robotSimType> -->
+        <!-- <bodyName>chassis</bodyName> -->
         <alwaysOn>true</alwaysOn>
         <updateRate>20</updateRate>
@@ -139,11 +140,11 @@
         <odometryTopic>odom</odometryTopic>
         <odometryFrame>odom</odometryFrame>
-        <robotBaseFrame>chassis</robotBaseFrame>
-        <publishWheelTF>false</publishWheelTF>
-        <publishOdom>false</publishOdom>
+        <robotBaseFrame>base_link</robotBaseFrame>
+        <publishWheelTF>true</publishWheelTF>
+        <publishOdom>true</publishOdom>
         <publishOdomTF>true</publishOdomTF>
-        <publishWheelJointState>false</publishWheelJointState>
-        <wheelAcceleration>0</wheelAcceleration>
-        <wheelTorque>5</wheelTorque>
+        <publishWheelJointState>true</publishWheelJointState>
+        <wheelAcceleration>1.0</wheelAcceleration>
+        <wheelTorque>20</wheelTorque>
         <odometrySource>world</odometrySource>
         <publishTf>1</publishTf>
@@ -159,12 +160,20 @@
     <gazebo reference="left_wheel">
       <selfCollide>true</selfCollide>
-      <mu1>0.2</mu1>
-      <mu2>0.2</mu2>
+      <mu1 value="1.0"/>
+      <mu2 value="1.0"/>
+      <kp  value="10000000.0" />
+      <kd  value="1.0" />
+      <fdir1 value="1 0 0"/>
+      <minDepth>0.02</minDepth>
       <material>Gazebo/Black</material>
     </gazebo>
     <gazebo reference="right_wheel">
       <selfCollide>true</selfCollide>
-      <mu1>0.2</mu1>
-      <mu2>0.2</mu2>
+      <mu1 value="1.0"/>
+      <mu2 value="1.0"/>
+      <kp  value="10000000.0" />
+      <kd  value="1.0" />
+      <fdir1 value="1 0 0"/>
+      <minDepth>0.02</minDepth>
       <material>Gazebo/Black</material>
     </gazebo>

File: lab2andDriver/drivers/universal_robot/ur_description/urdf/ur3_robot.urdf.xacro (robot description, xacro)
@@ -3,19 +3,19 @@
        name="ur3" >
   <xacro:arg name="transmission_hw_interface" default="hardware_interface/PositionJointInterface"/>
-  <!-- common stuff -->
+  <!-- common macros -->
   <xacro:include filename="$(find ur_description)/urdf/common.gazebo.xacro" />
+  <!-- ur3 macros-->
+  <xacro:include filename="$(find ur_description)/urdf/ur3.urdf.xacro" />
+  <!-- cart macros-->
+  <xacro:include filename="$(find ur_description)/urdf/myrobot.xacro" />
   <!-- ur3 -->
-  <xacro:include filename="$(find ur_description)/urdf/ur3.urdf.xacro" />
+  <xacro:ur3_robot prefix="" joint_limited="false"
+    transmission_hw_interface="$(arg transmission_hw_interface)" />
   <!-- cart -->
-  <xacro:include filename="$(find ur_description)/urdf/myrobot.xacro" />
-  <!-- arm -->
-  <xacro:ur3_robot prefix="" joint_limited="false"
-    transmission_hw_interface="$(arg transmission_hw_interface)"
-  />
   <xacro:cart_robot/>
   <joint name="ur3_cart_joint" type="fixed">
-    <parent link="chassis" />
-    <child link = "base_link" />
-    <origin xyz="0.0 0.0 0.05" rpy="0.0 0.0 0.0" />
+    <parent link="base_link" />
+    <child link = "chassis" />
+    <origin xyz="0.0 0.0 -0.05" rpy="0.0 0.0 0.0" />
   </joint>
 </robot>

Commit message: joint actuation confirmed

File: lab2andDriver/drivers/universal_robot/ur_description/urdf/myrobot.xacro (robot description, xacro)
@@ -136,5 +136,5 @@
         <wheelSeparation>0.4</wheelSeparation>
         <wheelDiameter>0.1</wheelDiameter>
-        <torque>20</torque>
+        <torque>40</torque>
         <commandTopic>cmd_vel</commandTopic>
         <odometryTopic>odom</odometryTopic>
@@ -146,5 +146,5 @@
         <publishWheelJointState>true</publishWheelJointState>
         <wheelAcceleration>1.0</wheelAcceleration>
-        <wheelTorque>20</wheelTorque>
+        <wheelTorque>40</wheelTorque>
         <odometrySource>world</odometrySource>
         <publishTf>1</publishTf>

File: lab2andDriver/drivers/universal_robot/ur_description/urdf/ur3_robot.urdf.xacro (robot description, xacro)
@@ -19,3 +19,10 @@
     <origin xyz="0.0 0.0 0.05" rpy="0.0 0.0 0.0" />
   </joint>
+<!--
+  <link name="world" />
+  <joint name="ur3_cart_joint_fix" type="fixed">
+    <parent link="world" />
+    <child link = "chassis" />
+    <origin xyz="0.0 0.0 0.0" rpy="0.0 0.0 0.0" />
+  </joint> -->
 </robot>

Commit message: added cart movement cvode

File: lab2andDriver/drivers/universal_robot/ur_description/urdf/myrobot.xacro (robot description, xacro)
@@ -8,5 +8,5 @@
       <pose>0 0 0.1 0 0 0</pose>
       <inertial>
-        <mass value="10.0"/>
+        <mass value="20.0"/>
         <origin xyz="0.0 0 0.1" rpy=" 0 0 0"/>
         <inertia
@@ -93,5 +93,5 @@
       <parent link="chassis"/>
       <axis xyz="0 1 0" rpy="0 0 0"/>
-      <!-- <limit velocity="100"/> -->
+      <limit effort="10000" velocity="10000"/>
       <joint_properties damping="0.0" friction="0.0"/>
     </joint>
@@ -101,5 +101,5 @@
       <parent link="chassis"/>
       <axis xyz="0 1 0" rpy="0 0 0"/>
-      <!-- <limit velocity="100"/> -->
+      <limit effort="10000" velocity="10000"/>
       <joint_properties damping="0.0" friction="0.0"/>
     </joint>
@@ -111,5 +111,5 @@
         <actuator name="leftMotor">
           <hardwareInterface>VelocityJointInterface</hardwareInterface>
-          <mechanicalReduction>10</mechanicalReduction>
+          <mechanicalReduction>1</mechanicalReduction>
         </actuator>
       </transmission>
@@ -121,5 +121,5 @@
         <actuator name="rightMotor">
           <hardwareInterface>VelocityJointInterface</hardwareInterface>
-          <mechanicalReduction>10</mechanicalReduction>
+          <mechanicalReduction>1</mechanicalReduction>
         </actuator>
       </transmission>
@@ -145,5 +145,5 @@
         <publishOdomTF>true</publishOdomTF>
         <publishWheelJointState>true</publishWheelJointState>
-        <wheelAcceleration>1.0</wheelAcceleration>
+        <wheelAcceleration>0.5</wheelAcceleration>
         <wheelTorque>40</wheelTorque>
         <odometrySource>world</odometrySource>
@@ -160,20 +160,12 @@
     <gazebo reference="left_wheel">
       <selfCollide>true</selfCollide>
-      <mu1 value="1.0"/>
-      <mu2 value="1.0"/>
-      <kp  value="10000000.0" />
-      <kd  value="1.0" />
-      <fdir1 value="1 0 0"/>
-      <minDepth>0.02</minDepth>
+      <mu1 value="20000.0"/>
+      <mu2 value="1000.0"/>
       <material>Gazebo/Black</material>
     </gazebo>
     <gazebo reference="right_wheel">
       <selfCollide>true</selfCollide>
-      <mu1 value="1.0"/>
-      <mu2 value="1.0"/>
-      <kp  value="10000000.0" />
-      <kd  value="1.0" />
-      <fdir1 value="1 0 0"/>
-      <minDepth>0.02</minDepth>
+      <mu1 value="20000.0"/>
+      <mu2 value="1000.0"/>
       <material>Gazebo/Black</material>
     </gazebo>

File: lab2andDriver/drivers/universal_robot/ur_description/urdf/ur3_robot.urdf.xacro (robot description, xacro)
@@ -19,9 +19,9 @@
     <origin xyz="0.0 0.0 0.05" rpy="0.0 0.0 0.0" />
   </joint>
-  <link name="world" />
+  <!-- <link name="world" />
   <joint name="ur3_cart_joint_fix" type="fixed">
     <parent link="world" />
     <child link = "chassis" />
     <origin xyz="0.0 0.0 0.0" rpy="0.0 0.0 0.0" />
-  </joint>
+  </joint> -->
 </robot>

Commit message: implemented translating prism

File: lab2andDriver/drivers/universal_robot/ur_description/urdf/myrobot.xacro (robot description, xacro)
@@ -6,8 +6,8 @@
   <xacro:macro name="cart_robot">
     <link name='chassis'>
-      <pose>0 0 0.1 0 0 0</pose>
+      <pose>0 0 0.075 0 0 0</pose>
       <inertial>
         <mass value="20.0"/>
-        <origin xyz="0.0 0 0.1" rpy=" 0 0 0"/>
+        <origin xyz="0.0 0 0.075" rpy=" 0 0 0"/>
         <inertia
             ixx="0.5" ixy="0" ixz="0"
@@ -18,5 +18,5 @@
       <collision name='collision'>
         <geometry>
-          <box size=".4 .2 .1"/>
+          <box size=".4 .2 .15"/>
         </geometry>
       </collision>
@@ -24,149 +24,21 @@
         <origin xyz="0 0 0" rpy=" 0 0 0"/>
         <geometry>
-          <box size=".4 .2 .1"/>
-        </geometry>
-      </visual>
-      <collision name='caster_collision'>
-        <origin xyz="-0.15 0 -0.05" rpy=" 0 0 0"/>
-        <geometry>
-          <sphere radius="0.05"/>
-        </geometry>
-      </collision>
-      <visual name='caster_visual'>
-        <origin xyz="-0.15 0 -0.05" rpy=" 0 0 0"/>
-        <geometry>
-          <sphere radius="0.05"/>
+          <box size=".4 .2 .15"/>
         </geometry>
       </visual>
     </link>
-    <link name="left_wheel">
-      <!--origin xyz="0.1 0.13 0.1" rpy="0 1.5707 1.5707"/-->
-      <collision name="collision">
-        <origin xyz="0 0 0" rpy="0 1.5707 1.5707"/>
-        <geometry>
-          <cylinder radius="0.1" length="0.05"/>
-        </geometry>
-      </collision>
-      <visual name="left_wheel_visual">
-        <origin xyz="0 0 0" rpy="0 1.5707 1.5707"/>
-        <geometry>
-          <cylinder radius="0.1" length="0.05"/>
-        </geometry>
-      </visual>
-      <inertial>
-        <origin xyz="0 0 0" rpy="0 1.5707 1.5707"/>
-        <mass value="5"/>
-        <cylinder_inertia m="5" r="0.1" h="0.05"/>
-        <inertia
-          ixx="1.0" ixy="0.0" ixz="0.0"
-          iyy="1.0" iyz="0.0"
-          izz="1.0"/>
-      </inertial>
-    </link>
-    <link name="right_wheel">
-      <!--origin xyz="0.1 -0.13 0.1" rpy="0 1.5707 1.5707"/-->
-      <collision name="collision">
-        <origin xyz="0 0 0" rpy="0 1.5707 1.5707"/>
-        <geometry>
-          <cylinder radius="0.1" length="0.05"/>
-        </geometry>
-      </collision>
-      <visual name="right_wheel_visual">
-        <origin xyz="0 0 0" rpy="0 1.5707 1.5707"/>
-        <geometry>
-          <cylinder radius="0.1" length="0.05"/>
-        </geometry>
-      </visual>
-      <inertial>
-        <origin xyz="0 0 0" rpy="0 1.5707 1.5707"/>
-        <mass value="5"/>
-        <cylinder_inertia m="5" r="0.1" h="0.05"/>
-        <inertia
-          ixx="1.0" ixy="0.0" ixz="0.0"
-          iyy="1.0" iyz="0.0"
-          izz="1.0"/>
-      </inertial>
-    </link>
-    <joint type="continuous" name="left_wheel_hinge">
-      <origin xyz="0.1 0.15 0" rpy="0 0 0"/>
-      <child link="left_wheel"/>
-      <parent link="chassis"/>
-      <axis xyz="0 1 0" rpy="0 0 0"/>
-      <limit effort="10000" velocity="10000"/>
-      <joint_properties damping="0.0" friction="0.0"/>
-    </joint>
-    <joint type="continuous" name="right_wheel_hinge">
-      <origin xyz="0.1 -0.15 0" rpy="0 0 0"/>
-      <child link="right_wheel"/>
-      <parent link="chassis"/>
-      <axis xyz="0 1 0" rpy="0 0 0"/>
-      <limit effort="10000" velocity="10000"/>
-      <joint_properties damping="0.0" friction="0.0"/>
-    </joint>
-    <transmission name="left_trans">
-        <type>transmission_interface/SimpleTransmission</type>
-        <joint name="left_wheel_hinge">
-          <hardwareInterface>hardware_interface/VelocityJointInterface</hardwareInterface>
-        </joint>
-        <actuator name="leftMotor">
-          <hardwareInterface>VelocityJointInterface</hardwareInterface>
-          <mechanicalReduction>1</mechanicalReduction>
-        </actuator>
-      </transmission>
-      <transmission name="right_trans">
-        <type>transmission_interface/SimpleTransmission</type>
-        <joint name="right_wheel_hinge">
-          <hardwareInterface>hardware_interface/VelocityJointInterface</hardwareInterface>
-        </joint>
-        <actuator name="rightMotor">
-          <hardwareInterface>VelocityJointInterface</hardwareInterface>
-          <mechanicalReduction>1</mechanicalReduction>
-        </actuator>
-      </transmission>
     <gazebo>
-      <plugin name="differential_drive_controller" filename="libgazebo_ros_diff_drive.so">
+      <plugin name="object_controller" filename="libgazebo_ros_planar_move.so">
         <robotNamespace>/cart_controller</robotNamespace>
-        <legacyMode>True</legacyMode>
-        <!-- <robotSimType>gazebo_ros_control/DefaultRobotHWSim</robotSimType> -->
-        <!-- <bodyName>chassis</bodyName> -->
-        <alwaysOn>true</alwaysOn>
-        <updateRate>20</updateRate>
-        <leftJoint>left_wheel_hinge</leftJoint>
-        <rightJoint>right_wheel_hinge</rightJoint>
-        <wheelSeparation>0.4</wheelSeparation>
-        <wheelDiameter>0.1</wheelDiameter>
-        <torque>40</torque>
         <commandTopic>cmd_vel</commandTopic>
         <odometryTopic>odom</odometryTopic>
         <odometryFrame>odom</odometryFrame>
-        <robotBaseFrame>base_link</robotBaseFrame>
-        <publishWheelTF>true</publishWheelTF>
-        <publishOdom>true</publishOdom>
-        <publishOdomTF>true</publishOdomTF>
-        <publishWheelJointState>true</publishWheelJointState>
-        <wheelAcceleration>0.5</wheelAcceleration>
-        <wheelTorque>40</wheelTorque>
-        <odometrySource>world</odometrySource>
-        <publishTf>1</publishTf>
-        <rosDebugLevel>na</rosDebugLevel>
+        <odometryRate>20.0</odometryRate>
+        <robotBaseFrame>chassis</robotBaseFrame>
       </plugin>
     </gazebo>
     <gazebo reference="chassis">
       <selfCollide>true</selfCollide>
-      <mu1>0.0</mu1>
-      <mu2>0.0</mu2>
       <material>Gazebo/Orange</material>
-    </gazebo>
-    <gazebo reference="left_wheel">
-      <selfCollide>true</selfCollide>
-      <mu1 value="20000.0"/>
-      <mu2 value="1000.0"/>
-      <material>Gazebo/Black</material>
-    </gazebo>
-    <gazebo reference="right_wheel">
-      <selfCollide>true</selfCollide>
-      <mu1 value="20000.0"/>
-      <mu2 value="1000.0"/>
-      <material>Gazebo/Black</material>
     </gazebo>
   </xacro:macro>

File: lab2andDriver/drivers/universal_robot/ur_description/urdf/ur3_robot.urdf.xacro (robot description, xacro)
@@ -17,11 +17,5 @@
     <parent link="chassis" />
     <child link = "base_link" />
-    <origin xyz="0.0 0.0 0.05" rpy="0.0 0.0 0.0" />
+    <origin xyz="0.0 0.0 0.075" rpy="0.0 0.0 0.0" />
   </joint>
-  <!-- <link name="world" />
-  <joint name="ur3_cart_joint_fix" type="fixed">
-    <parent link="world" />
-    <child link = "chassis" />
-    <origin xyz="0.0 0.0 0.0" rpy="0.0 0.0 0.0" />
-  </joint> -->
 </robot>

Commit message: final push

File: lab2andDriver/drivers/universal_robot/ur_description/urdf/myrobot.xacro (robot description, xacro)
@@ -8,5 +8,5 @@
       <pose>0 0 0.075 0 0 0</pose>
       <inertial>
-        <mass value="20.0"/>
+        <mass value="150.0"/>
         <origin xyz="0.0 0 0.075" rpy=" 0 0 0"/>
         <inertia
@@ -18,5 +18,5 @@
       <collision name='collision'>
         <geometry>
-          <box size=".4 .2 .15"/>
+          <box size=".4 .4 .15"/>
         </geometry>
       </collision>
@@ -24,5 +24,5 @@
         <origin xyz="0 0 0" rpy=" 0 0 0"/>
         <geometry>
-          <box size=".4 .2 .15"/>
+          <box size=".4 .4 .15"/>
         </geometry>
       </visual>
